Commit message: matched sim to actual robot

File: desc/gazebo_sim_control.xacro (robot description, xacro)
@@ -5,6 +5,6 @@
             <left_joint>left_wheel_joint</left_joint>
             <right_joint>right_wheel_joint</right_joint>
-            <wheel_separation>0.35</wheel_separation>
-            <wheel_diamater>0.1</wheel_diamater>
+            <wheel_separation>0.1827</wheel_separation>
+            <wheel_diamater>0.066</wheel_diamater>
             <max_wheel_torque>200</max_wheel_torque>
             <max_wheel_acceleration>10</max_wheel_acceleration>

File: desc/gz_depth_camera_control.xacro (robot description, xacro)
@@ -4,5 +4,5 @@
         <parent link="chassis"/>
         <child link="camera_link"/>
-        <origin xyz="0.305 0 0.08" rpy="0 0 0"/>
+        <origin xyz="0.1 0 0.018" rpy="0 0 0"/>
     </joint>
     <link name="camera_link">
@@ -10,16 +10,16 @@
             <origin xyz='0 0 0'/>
             <geometry>
-                <box size='0.01 0.03 0.03'/>
+                <box size='0.02 0.085 0.024'/>
             </geometry>
-            <material name='red'/>
+            <material name='black'/>
         </visual>
         <collision>
             <geometry>
-                <cylinder radius='0.05' length='0.04'/>
+                <box size='0.02 0.085 0.024'/>
             </geometry>
         </collision>
-        <xacro:cylinder_moi mass='0.5' r='0.05' l='0.04'>
+        <xacro:cuboid_moi mass='0.023' l='0.02' b='0.085' h='0.024'>
             <origin xyz='0 0 0' rpy='0 0 0'/>
-        </xacro:cylinder_moi>
+        </xacro:cuboid_moi>7
     </link>
     <joint name="optical_joint" type="fixed">

File: desc/lidar_control.xacro (robot description, xacro)
@@ -4,5 +4,5 @@
         <parent link="chassis"/>
         <child link="lidar_link"/>
-        <origin xyz="0.1 0 0.175" rpy="0 0 0"/>
+        <origin xyz="0 0 0.054" rpy="0 0 0"/>
     </joint>
     <link name="lidar_link">
@@ -10,14 +10,14 @@
             <origin xyz='0 0 0'/>
             <geometry>
-                <cylinder radius='0.05' length='0.04'/>
+                <cylinder radius='0.02' length='0.04'/>
             </geometry>
-            <material name='red'/>
+            <material name='black'/>
         </visual>
         <collision>
             <geometry>
-                <cylinder radius='0.05' length='0.04'/>
+                <cylinder radius='0.02' length='0.04'/>
             </geometry>
         </collision>
-        <xacro:cylinder_moi mass='0.5' r='0.05' l='0.04'>
+        <xacro:cylinder_moi mass='0.045' r='0.02' l='0.04'>
             <origin xyz='0 0 0' rpy='0 0 0'/>
         </xacro:cylinder_moi>

File: desc/materials.xacro (robot description, xacro)
@@ -16,3 +16,6 @@
         <color rgba='0 0 1 1'/>
     </material>
+	<material name='purple'>
+        <color rgba='0.5 0 0.5 1'/>
+    </material>
 </robot>

File: desc/robot_base.xacro (robot description, xacro)
@@ -8,22 +8,22 @@
         <parent link='base_link'/>
         <child link='chassis'/>
-        <origin xyz='-0.1 0 0'/>
+        <origin xyz='0.02 0 0.014'/>
     </joint>
     <link name='chassis'>
         <visual>
-            <origin xyz='0.15 0 0.075'/>
+            <origin xyz='0 0 0'/>
             <geometry>
-                <box size='0.3 0.3 0.15'/>
+                <box size='0.18 0.18 0.068'/>
             </geometry>
-            <material name='black'/>
+            <material name='purple'/>
         </visual>
         <collision>
-            <origin xyz='0.15 0 0.075'/>
+            <origin xyz='0 0 0'/>
             <geometry>
-                <box size='0.3 0.3 0.15'/>
+                <box size='0.18 0.18 0.068'/>
             </geometry>
         </collision>
-        <xacro:cuboid_moi mass='0.5' l='0.3' b='0.3' h='0.15'>
-            <origin xyz='0.15 0 0.075' rpy='0 0 0'/>
+        <xacro:cuboid_moi mass='1.0635' l='0.18' b='0.18' h='0.068'>
+            <origin xyz='0 0 0' rpy='0 0 0'/>
         </xacro:cuboid_moi>
     </link>
@@ -31,22 +31,23 @@
         <parent link='base_link'/>
         <child link='left_wheel'/>
-        <origin xyz='0 0.17 0' rpy='-${pi/2} 0 0'/>
+        <origin xyz='0 0.09 0' rpy='-${pi/2} 0 0'/>
         <axis xyz='0 0 1'/>
     </joint>
     <link name='left_wheel'>
         <visual>
-            <origin xyz='0 0 0'/>
+            <origin xyz='0 0 0.0135'/>
             <geometry>
-                <cylinder radius='0.05' length='0.04'/>
+                <cylinder radius='0.033' length='0.027'/>
             </geometry>
-            <material name='grey'/>
+            <material name='blue'/>
         </visual>
         <collision>
+			<origin xyz='0 0 0.0135'/>
             <geometry>
-                <cylinder radius='0.05' length='0.04'/>
+                <cylinder radius='0.033' length='0.027'/>
             </geometry>
         </collision>
-        <xacro:cylinder_moi mass='0.5' r='0.05' l='0.04'>
-            <origin xyz='0 0 0' rpy='0 0 0'/>
+        <xacro:cylinder_moi mass='0.033' r='0.033' l='0.027'>
+            <origin xyz='0 0 0.0135' rpy='0 0 0'/>
         </xacro:cylinder_moi>
     </link>
@@ -54,28 +55,29 @@
         <parent link='base_link'/>
         <child link='right_wheel'/>
-        <origin xyz='0 -0.17 0' rpy='${pi/2} 0 0'/>
+        <origin xyz='0 -0.09 0' rpy='${pi/2} 0 0'/>
         <axis xyz='0 0 -1'/>
     </joint>
     <link name='right_wheel'>
         <visual>
-            <origin xyz='0 0 0'/>
+            <origin xyz='0 0 0.0135'/>
             <geometry>
-                <cylinder radius='0.05' length='0.04'/>
+                <cylinder radius='0.033' length='0.027'/>
             </geometry>
-            <material name='grey'/>
+            <material name='blue'/>
         </visual>
         <collision>
+			<origin xyz='0 0 0.0135'/>
             <geometry>
-                <cylinder radius='0.05' length='0.04'/>
+                <cylinder radius='0.033' length='0.027'/>
             </geometry>
         </collision>
-        <xacro:cylinder_moi mass='0.5' r='0.05' l='0.04'>
-            <origin xyz='0 0 0' rpy='0 0 0'/>
+        <xacro:cylinder_moi mass='0.033' r='0.033' l='0.027'>
+            <origin xyz='0 0 0.0135' rpy='0 0 0'/>
         </xacro:cylinder_moi>
     </link>
     <joint name='caster_wheel_joint' type='fixed'>
-        <parent link='chassis'/>
+        <parent link='base_link'/>
         <child link='caster_wheel'/>
-        <origin xyz='0.25 0 0'/>
+        <origin xyz='0.085 0 -0.02'/>
     </joint>
     <link name='caster_wheel'>
@@ -83,14 +85,14 @@
             <origin xyz='0 0 0'/>
             <geometry>
-                <sphere radius='0.05'/>
+                <sphere radius='0.0085'/>
             </geometry>
-            <material name='grey'/>
+            <material name='blue'/>
         </visual>
         <collision>
             <geometry>
-                <sphere radius='0.05'/>
+                <sphere radius='0.0085'/>
             </geometry>
         </collision>
-        <xacro:sphere_moi mass='0.5' r='0.05'>
+        <xacro:sphere_moi mass='0.043' r='0.0085'>
             <origin xyz='0 0 0' rpy='0 0 0'/>
         </xacro:sphere_moi>
